Commit message: feat: update robot design

File: my_robot/urdf/my_robot.xacro (robot description, xacro)
@@ -30,8 +30,20 @@
             />
         </inertial>
+        <!--<collision name='collision'>
+            <origin xyz="0 0 0" rpy="0 0 0"/>
+            <geometry>
+                <box size=".8 .8 .1"/>
+            </geometry>
+        </collision>
+        <visual name='chassis_visual'>
+            <origin xyz = "0 0 0" rpy = "0 0 0"/>
+            <geometry>
+                <box size=".8 .8 .1"/>
+            </geometry>
+        </visual>-->
         <collision name='collision'>
             <origin xyz="0 0 0" rpy="0 0 0"/>
             <geometry>
-                <box size=".4 .2 .1"/>
+                <cylinder radius="0.4" length="0.1"/>
             </geometry>
         </collision>
@@ -39,34 +51,34 @@
             <origin xyz = "0 0 0" rpy = "0 0 0"/>
             <geometry>
-                <box size=".4 .2 .1"/>
+                <cylinder radius="0.4" length="0.1"/>
             </geometry>
         </visual>
         <collision name = 'back_caster_collision'>
-            <origin xyz = "-0.15 0 -0.05" rpy=" 0 0 0"/>
-            <geometry>
-                <sphere radius="0.0499"/>
+            <origin xyz = "-0.3 0 -0.1" rpy=" 0 0 0"/>
+            <geometry>
+                <sphere radius="0.099"/>
             </geometry>
         </collision>
         <visual name='back_caster_visual'>
-            <origin xyz = "-0.15 0 -0.05" rpy=" 0 0 0"/>
-            <geometry>
-                <sphere radius="0.05"/>
+            <origin xyz = "-0.3 0 -0.1" rpy=" 0 0 0"/>
+            <geometry>
+                <sphere radius="0.1"/>
             </geometry>
         </visual>
         <collision name = 'front_caster_collision'>
-            <origin xyz = "0.15 0 -0.05" rpy=" 0 0 0"/>
-            <geometry>
-                <sphere radius="0.0499"/>
+            <origin xyz = "0.3 0 -0.1" rpy=" 0 0 0"/>
+            <geometry>
+                <sphere radius="0.099"/>
             </geometry>
         </collision>
         <visual name='front_caster_visual'>
-            <origin xyz = "0.15 0 -0.05" rpy=" 0 0 0"/>
-            <geometry>
-                <sphere radius="0.05"/>
+            <origin xyz = "0.3 0 -0.1" rpy=" 0 0 0"/>
+            <geometry>
+                <sphere radius="0.1"/>
             </geometry>
         </visual>
     </link>
     <gazebo reference="chassis">
-        <material>Gazebo/Blue</material>
+        <material>Gazebo/Green</material>
     </gazebo>
     <link name='left_wheel'>
@@ -83,5 +95,5 @@
             <origin xyz = "0.0 0 0.0" rpy=" 0 1.5707 1.5707"/>
             <geometry>
-                <cylinder radius="0.1" length="0.05"/>
+                <cylinder radius="0.2" length="0.05"/>
             </geometry>
         </collision>
@@ -89,10 +101,10 @@
             <origin xyz = "0.0 0 0.0" rpy=" 0 1.5707 1.5707"/>
             <geometry>
-                <cylinder radius="0.1" length="0.05"/>
+                <cylinder radius="0.2" length="0.05"/>
             </geometry>
         </visual>
     </link>
     <gazebo reference="left_wheel">
-        <material>Gazebo/Green</material>
+        <material>Gazebo/Black</material>
     </gazebo>
     <link name='right_wheel'>
@@ -109,5 +121,5 @@
             <origin xyz = "0.0 0 0.0" rpy=" 0 1.5707 1.5707"/>
             <geometry>
-                <cylinder radius="0.1" length="0.05"/>
+                <cylinder radius="0.2" length="0.05"/>
             </geometry>
         </collision>
@@ -115,13 +127,13 @@
             <origin xyz = "0.0 0 0.0" rpy=" 0 1.5707 1.5707"/>
             <geometry>
-                <cylinder radius="0.1" length="0.05"/>
+                <cylinder radius="0.2" length="0.05"/>
             </geometry>
         </visual>
     </link>
     <gazebo reference="right_wheel">
-        <material>Gazebo/Green</material>
+        <material>Gazebo/Black</material>
     </gazebo>
     <joint type = "continuous" name = "left_wheel_hinge">
-        <origin xyz="0 0.15 0" rpy="0 0 0"/>
+        <origin xyz="0 0.45 0" rpy="0 0 0"/>
         <child link="left_wheel"/>
         <parent link="chassis"/>
@@ -131,5 +143,5 @@
     </joint>
     <joint type = "continuous" name = "right_wheel_hinge">
-        <origin xyz="0 -0.15 0" rpy="0 0 0"/>
+        <origin xyz="0 -0.45 0" rpy="0 0 0"/>
         <child link="right_wheel"/>
         <parent link="chassis"/>
@@ -163,8 +175,8 @@
     </link>
     <gazebo reference="camera">
-        <material>Gazebo/Red</material>
+        <material>Gazebo/Yellow</material>
     </gazebo>
     <joint type = "fixed" name = "camera_joint">
-        <origin xyz="0.2 0 0" rpy="0 0 0"/>
+        <origin xyz="0.4 0 0" rpy="0 0 0"/>
         <child link="camera"/>
         <parent link="chassis"/>
@@ -195,5 +207,5 @@
     </link>
     <joint type = "fixed" name = "hokuyo_joint">
-        <origin xyz="0.15 0 0.1" rpy="0 0 0"/>
+        <origin xyz="0.35 0 0.1" rpy="0 0 0"/>
         <child link="hokuyo"/>
         <parent link="chassis"/>

Commit message: feat: add a shovel to the robot, enable ball catch

File: my_robot/urdf/my_robot.xacro (robot description, xacro)
@@ -10,7 +10,19 @@
         <color rgba="0 0.8 0 1"/>
     </material>
+    <material name="white">
+        <color rgba="1.0 1.0 1.0 1"/>
+    </material>
     <!-- Include plugins-->
     <xacro:include filename="$(find my_robot)/urdf/my_robot.gazebo" />
-    <!-- link and joints definition -->
+    <!-- Include arm definition file-->
+    <xacro:include filename="$(find my_robot)/urdf/arm.xacro" />
+    <!-- Include ball container file -->
+    <xacro:include filename="$(find my_robot)/urdf/ball_container.xacro" />
+    <!-- create the left and right arm-->
+    <arm lr="left" tY =  "-1" />
+    <arm lr="right" tY = "1" />
+    <!-- create ball container-->
+    <ball_container/>
+    <!-- link and joints definition of the robot chassis and wheel-->
     <link name="robot_footprint"></link>
     <joint name="robot_footprint_joint" type="fixed">
